Commit message: try different joint angles for the laser

File: src/my_robot/urdf/my_robot.xacro (robot description, xacro)
@@ -212,5 +212,5 @@
         </link>
         <joint type="fixed" name="hokuyo_joint_back">
-            <origin xyz="-0.15 0 0.1" rpy="0 0 3.14" />
+            <origin xyz="-0.15 0 0.1" rpy="0 0 0" />
             <parent link="chassis" />
             <child link="hokuyo_back" />

Commit message: add new robot model

File: src/my_robot/urdf/my_robot.xacro (robot description, xacro)
@@ -1,219 +1,186 @@
-<?xml version="1.0" encoding="UTF-8"?>
-<robot name="my_robot" xmlns:xacro="https://www.ros.org/wiki/xacro" >
-<xacro:include filename="$(find my_robot)/urdf/my_robot.gazebo" />
-    <gazebo reference="left_wheel">
-        <material>Gazebo/Black</material>
-    </gazebo>
-    <gazebo reference="right_wheel">
-        <material>Gazebo/Black</material>
-    </gazebo>
-    <gazebo reference="chassis">
-        <material>Gazebo/Yellow</material>
-    </gazebo>
-    <gazebo reference="camera">
-        <material>Gazebo/Grey</material>
-    </gazebo>
-        <link name="robot_footprint"></link>
-        <joint name="robot_footprint" type="fixed">
-            <origin xyz="0 0 0" rpy="0 0 0" />
-            <parent link="robot_footprint" />
-            <child link="chassis" />
-        </joint>
-        <link name="chassis">
-            <pose>0 0 0.1 0 0 0</pose>
-            <inertial>
-                <mass value="15.0"/>
-                <origin xyz="0.0 0 0" rpy=" 0 0 0"/>
-                <inertia
-                    ixx="0.1" ixy="0" ixz="0"
-                    iyy="0.1" iyz="0"
-                    izz="0.1"
-                />
-              </inertial>
-              <collision name='collision'>
-                <origin xyz="0 0 0" rpy=" 0 0 0"/>
-                <geometry>
-                  <box size=".4 .2 .1"/>
-                </geometry>
-              </collision>
-              <visual name='chassis_visual'>
-                <origin xyz="0 0 0" rpy=" 0 0 0"/>
-                <geometry>
-                  <box size=".4 .2 .1"/>
-                </geometry>
-              </visual>
-              <collision name='back_caster_collision'>
-                <origin xyz="-0.15 0 -0.05" rpy=" 0 0 0"/>
-                <geometry>
-                  <sphere radius="0.0499"/>
-                </geometry>
-              </collision>
-              <visual name='back_caster_visual'>
-                <origin xyz="-0.15 0 -0.05" rpy=" 0 0 0"/>
-                <geometry>
-                  <sphere radius="0.05"/>
-                </geometry>
-              </visual>
-              <collision name='front_caster_collision'>
-                <origin xyz="0.15 0 -0.05" rpy=" 0 0 0"/>
-                <geometry>
-                  <sphere radius="0.0499"/>
-                </geometry>
-              </collision>
-              <visual name='front_caster_visual'>
-                <origin xyz="0.15 0 -0.05" rpy=" 0 0 0"/>
-                <geometry>
-                  <sphere radius="0.05"/>
-                </geometry>
-              </visual>
-        </link>
-        <joint type="continuous" name="left_wheel_hinge" >
-            <origin xyz="0 0.15 0" rpy="0 0 0" />
-            <child link="left_wheel" />
-            <parent link="chassis" />
-            <axis xyz="0 1 0" rpy="0 0 0" />
-            <limit effort="10000" velocity="1000" />
-            <dynamics damping="1.0" friction="1.0" />
-        </joint>
-        <link name="left_wheel">
-            <visual name="left_wheel_visual">
-                <geometry>
-                    <cylinder radius='0.1' length='0.05'></cylinder>
-                </geometry>
-                <origin xyz="0 0 0" rpy="0 1.5708 1.5708"/>
-            </visual>
-            <collision name="left_wheel_collision">
-                <geometry>
-                    <cylinder radius='0.1' length='0.05'></cylinder>
-                </geometry>
-                <origin xyz="0 0 0" rpy="0 1.5708 1.5708"/>
-            </collision>
-            <inertial>
-                <mass value="5"/>
-                <origin xyz="0 0 0" rpy="0 1.5708 1.5708" />
-                <inertia
-                ixx="0.1" ixy="0" ixz="0"
-                iyy="0.1" iyz="0"
-                izz="0.1"
-                />
-            </inertial>
-        </link>
-        <link name="right_wheel">
-            <visual name="right_wheel_visual">
-                <geometry>
-                    <cylinder radius='0.1' length='0.05'></cylinder>
-                </geometry>
-                <origin xyz="0 0 0" rpy="0 1.5708 1.5708"/>
-            </visual>
-            <collision name="right_wheel_collision">
-                <geometry>
-                    <cylinder radius='0.1' length='0.05'></cylinder>
-                </geometry>
-                <origin xyz="0 0 0" rpy="0 1.5708 1.5708"/>
-            </collision>
-            <inertial>
-                <mass value="5"/>
-                <origin xyz="0 0 0" rpy="0 1.5708 1.5708" />
-                <inertia
-                ixx="0.1" ixy="0" ixz="0"
-                iyy="0.1" iyz="0"
-                izz="0.1"
-                />
-            </inertial>
-        </link>
-        <joint type="continuous" name="right_wheel_hinge" >
-            <origin xyz="0 -0.15 0" rpy="0 0 0" />
-            <child link="right_wheel" />
-            <parent link="chassis" />
-            <axis xyz="0 1 0" rpy="0 0 0" />
-            <limit effort="10000" velocity="1000" />
-            <dynamics damping="1.0" friction="1.0" />
-        </joint>
-        <link name="camera">
-            <visual name="camera_visual">
-                <geometry>
-                    <box size="0.05 0.05 0.05"/>
-                </geometry>
-                <origin xyz="0 0 0" rpy="0 0 0" />
-            </visual>
-            <collision name="camera_collision">
-                <geometry>
-                    <box size="0.05 0.05 0.05"/>
-                </geometry>
-                <origin xyz="0 0 0" rpy="0 0 0" />
-            </collision>
-            <inertial>
-                <mass value="0.1"/>
-                <origin xyz="0 0 0" rpy="0 0 0" />
-                <inertia
-                ixx="1e-6" ixy="0" ixz="0"
-                iyy="1e-6" iyz="0"
-                izz="1e-6"
-                />
-            </inertial>
-        </link>
-        <joint type="fixed" name="camera_joint">
-            <origin xyz=" 0.2 0 0" rpy="0 0 0" />
-            <child link="camera"/>
-            <parent link="chassis" />
-            <axis xyz=" 0 1 0 " rpy="0 0 0" />
-        </joint>
-        <link name="hokuyo_front">
-            <visual name="hokuyo_visual_front">
-                <geometry>
-                    <mesh filename="package://my_robot/meshes/hokuyo.dae" />
-                </geometry>
-                <origin xyz="0 0 0" rpy="0 0 0" />
-            </visual>
-            <collision name="camera_collision">
-                <geometry>
-                    <box size="0.1 0.1 0.1"/>
-                </geometry>
-                <origin xyz="0 0 0" rpy="0 0 0" />
-            </collision>
-            <inertial>
-                <mass value="1e-5"/>
-                <origin xyz="0 0 0" rpy="0 0 0" />
-                <inertia
-                ixx="1e-6" ixy="0" ixz="0"
-                iyy="1e-6" iyz="0"
-                izz="1e-6"
-                />
-            </inertial>
-        </link>
-        <joint type="fixed" name="hokuyo_joint_front">
-            <origin xyz="0.15 0 0.1" rpy="0 0 0" />
-            <parent link="chassis" />
-            <child link="hokuyo_front" />
-            <axis xyz="0 1 0" rpy="0 0 0" />
-        </joint>
-         <link name="hokuyo_back">
-            <visual name="hokuyo_visual_back">
-                <geometry>
-                    <mesh filename="package://my_robot/meshes/hokuyo.dae" />
-                </geometry>
-                <origin xyz="0 0 0" rpy="0 0 0" />
-            </visual>
-            <collision name="camera_collision">
-                <geometry>
-                    <box size="0.1 0.1 0.1"/>
-                </geometry>
-                <origin xyz="0 0 0" rpy="0 0 0" />
-            </collision>
-            <inertial>
-                <mass value="1e-5"/>
-                <origin xyz="0 0 0" rpy="0 0 0" />
-                <inertia
-                ixx="1e-6" ixy="0" ixz="0"
-                iyy="1e-6" iyz="0"
-                izz="1e-6"
-                />
-            </inertial>
-        </link>
-        <joint type="fixed" name="hokuyo_joint_back">
-            <origin xyz="-0.15 0 0.1" rpy="0 0 0" />
-            <parent link="chassis" />
-            <child link="hokuyo_back" />
-            <axis xyz="0 1 0" rpy="0 0 0" />
-        </joint>
-</robot>
+<?xml version='1.0'?>
+<robot name="my_robot" xmlns:xacro="http://www.ros.org/wiki/xacro">
+  <xacro:include filename="$(find my_robot)/urdf/my_robot.gazebo" />
+  <link name="robot_footprint"></link>
+  <joint name="robot_footprint_joint" type="fixed">
+    <origin xyz="0 0 0" rpy="0 0 0" />
+    <parent link="robot_footprint"/>
+    <child link="chassis" />
+  </joint>
+  <link name='chassis'>
+    <pose>0 0 0.1 0 0 0</pose>
+    <inertial>
+      <mass value="15.0"/>
+      <origin xyz="0.0 0 0" rpy=" 0 0 0"/>
+      <inertia
+              ixx="0.1" ixy="0" ixz="0"
+              iyy="0.1" iyz="0"
+              izz="0.1"
+      />
+    </inertial>
+    <collision name='collision'>
+      <origin xyz="0 0 0" rpy=" 0 0 0"/>
+      <geometry>
+        <box size=".4 .2 .1"/>
+      </geometry>
+    </collision>
+    <visual name='chassis_visual'>
+      <origin xyz="0 0 0" rpy=" 0 0 0"/>
+      <geometry>
+        <box size=".4 .2 .1"/>
+      </geometry>
+    </visual>
+    <collision name='back_caster_collision'>
+      <origin xyz="-0.15 0 -0.05" rpy=" 0 0 0"/>
+      <geometry>
+        <sphere radius="0.0499"/>
+      </geometry>
+    </collision>
+    <visual name='back_caster_visual'>
+      <origin xyz="-0.15 0 -0.05" rpy=" 0 0 0"/>
+      <geometry>
+        <sphere radius="0.05"/>
+      </geometry>
+    </visual>
+    <collision name='front_caster_collision'>
+      <origin xyz="0.15 0 -0.05" rpy=" 0 0 0"/>
+      <geometry>
+        <sphere radius="0.0499"/>
+      </geometry>
+    </collision>
+    <visual name='front_caster_visual'>
+      <origin xyz="0.15 0 -0.05" rpy=" 0 0 0"/>
+      <geometry>
+        <sphere radius="0.05"/>
+      </geometry>
+    </visual>
+  </link>
+  <!-- Add two wheels -->
+  <link name="left_wheel">
+    <inertial>
+      <origin xyz="0 0 0" rpy="0 1.5707 1.5707"/>
+      <mass value="5"/>
+      <inertia
+              ixx="0.1" ixy="0" ixz="0"
+              iyy="0.1" iyz="0" izz="0.1"
+      />
+    </inertial>
+    <collision>
+      <origin xyz="0 0 0" rpy="0 1.5707 1.5707"/>
+      <geometry>
+        <cylinder radius="0.1" length="0.05"/>
+      </geometry>
+    </collision>
+    <visual>
+      <origin xyz="0 0 0" rpy="0 1.5707 1.5707"/>
+      <geometry>
+        <cylinder radius="0.1" length="0.05"/>
+      </geometry>
+    </visual>
+  </link>
+  <link name="right_wheel">
+    <inertial>
+      <origin xyz="0 0 0" rpy="0 1.5707 1.5707"/>
+      <mass value="5"/>
+      <inertia
+              ixx="0.1" ixy="0" ixz="0"
+              iyy="0.1" iyz="0" izz="0.1"
+      />
+    </inertial>
+    <collision>
+      <origin xyz="0 0 0" rpy="0 1.5707 1.5707"/>
+      <geometry>
+        <cylinder radius="0.1" length="0.05"/>
+      </geometry>
+    </collision>
+    <visual>
+      <origin xyz="0 0 0" rpy="0 1.5707 1.5707"/>
+      <geometry>
+        <cylinder radius="0.1" length="0.05"/>
+      </geometry>
+    </visual>
+  </link>
+  <joint name="left_wheel_hinge" type="continuous">
+    <origin xyz="0 0.125 0" rpy="0 0 0"/>
+    <child link="left_wheel"/>
+    <parent link="chassis"/>
+    <axis xyz="0 1 0" rpy="0 0 0"/>
+    <limit effort="10000" velocity="1000"/>
+    <dynamics damping="1.0" friction="1.0"/>
+  </joint>
+  <joint name="right_wheel_hinge" type="continuous">
+    <origin xyz="0 -0.125 0" rpy="0 0 0"/>
+    <child link="right_wheel"/>
+    <parent link="chassis"/>
+    <axis xyz="0 1 0" rpy="0 0 0"/>
+    <limit effort="10000" velocity="1000"/>
+    <dynamics damping="1.0" friction="1.0"/>
+  </joint>
+  <!-- Add camera -->
+  <link name="camera">
+    <origin xyz="0 0 0" rpy="0 0 0" />
+    <inertial>
+      <mass value="0.1"/>
+      <inertia
+              ixx="1e-6" ixy="0" ixz="0"
+              iyy="1e-6" iyz="0" izz="1e-6"
+      />
+    </inertial>
+    <collision>
+      <geometry>
+        <box size="0.05 0.05 0.05"/>
+      </geometry>
+    </collision>
+    <visual>
+      <geometry>
+        <box size="0.05 0.05 0.05"/>
+      </geometry>
+    </visual>
+  </link>
+  <joint name="camera_joint" type="fixed">
+    <axis xyz="0 1 0"/>
+    <origin xyz="0.2 0 0" rpy="0 0 0" />
+    <parent link="chassis"/>
+    <child link="camera" />
+  </joint>
+  <!-- Add Lidar -->
+  <link name="hokuyo">
+    <origin xyz="0 0 0" rpy="0 0 0" />
+    <inertial>
+      <mass value="1e-5"/>
+      <inertia
+              ixx="1e-6" ixy="0" ixz="0"
+              iyy="1e-6" iyz="0" izz="1e-6"
+      />
+    </inertial>
+    <collision>
+      <geometry>
+        <box size=".1 .1 .1"/>
+      </geometry>
+    </collision>
+    <visual>
+      <geometry>
+        <mesh filename="package://my_robot/meshes/hokuyo.dae"/>
+      </geometry>
+    </visual>
+  </link>
+  <joint name="hokuyo_joint" type="fixed">
+    <axis xyz="0 1 0"/>
+    <origin xyz="0.15 0 0.1" rpy="0 0 0" />
+    <parent link="chassis"/>
+    <child link="hokuyo" />
+  </joint>
+  <!-- Color the components -->
+  <gazebo reference="chassis">
+    <material>Gazebo/Orange</material>
+  </gazebo>
+  <gazebo reference="left_wheel">
+    <material>Gazebo/Green</material>
+  </gazebo>
+  <gazebo reference="right_wheel">
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
Commit message: Add imu and gps sensors to the robot model

File: src/my_robot/urdf/my_robot.xacro (robot description, xacro)
@@ -2,4 +2,5 @@
 <robot name="my_robot" xmlns:xacro="http://www.ros.org/wiki/xacro">
   <xacro:include filename="$(find my_robot)/urdf/my_robot.gazebo" />
+  <xacro:property name="dummy_inertia" value="1e-09"/>
   <link name="robot_footprint"></link>
   <joint name="robot_footprint_joint" type="fixed">
@@ -171,4 +172,32 @@
     <child link="hokuyo" />
   </joint>
+  <!-- add imu and gps -->
+  <link name="navsat_link">
+    <origin xyz="0 0 0" rpy="0 0 0" />
+    <visual>
+      <geometry>
+        <cylinder radius="0.026" length="0.016" />
+      </geometry>
+      <origin xyz="0 0 0.008" />
+      <material name="black" />
+    </visual>
+  </link>
+  <joint name="navsat_joint" type="fixed">
+    <parent link="chassis" />
+    <child link="navsat_link" />
+    <origin xyz="-0.10 0.0 0.05" />
+  </joint>
+  <!-- imu -->
+  <link name="imu_link">
+    <inertial>
+      <mass value="0.001"/>
+      <origin xyz="0 0 0" rpy="0 0 0"/>
+      <inertia ixx="${dummy_inertia}" ixy="0.0" ixz="0.0" iyy="${dummy_inertia}" iyz="0.0" izz="${dummy_inertia}"/>
+    </inertial>
+  </link>
+  <joint name="imu_joint" type="fixed">
+    <parent link="chassis" />
+    <child link="imu_link" />
+  </joint>
   <!-- Color the components -->
   <gazebo reference="chassis">
