Commit message: Port robot_description to ROS2 Jazzy + Gazebo Harmonic
- package.xml: catkin → ament_cmake (format 3), add ros_gz_sim/bridge deps
- CMakeLists.txt: catkin boilerplate → clean ament_cmake with install targets
- urdf/automaton.gazebo: Gazebo Classic plugins → Gazebo Harmonic systems
    DiffDrive, JointStatePublisher; IMU/ground-truth blocks kept as comments
- urdf/laser.urdf.xacro: libgazebo_ros_laser.so → gpu_lidar sensor type,
    topic-based so ros_gz_bridge handles ROS2 publishing
- worlds/automaton_world.sdf: custom world loading Physics, Sensors, Imu,
    SceneBroadcaster systems (required for gpu_lidar to work)
- launch/description.launch.py: standalone RViz2 model viewer with
    joint_state_publisher_gui (replaces description.launch XML)
- launch/gazebo.launch.py: full sim stack — gz_sim, robot spawn, ros_gz_bridge
    for clock/cmd_vel/odom/tf/laser/joint_states, RViz2
- rviz_config/automaton.rviz: RViz2 format — rviz/ → rviz_default_plugins/,
    RobotModel uses /robot_description topic, LaserScan QoS configured

File: src/robot_description/urdf/laser.urdf.xacro (robot description, xacro)
@@ -1,19 +1,31 @@
 <?xml version="1.0"?>
 <robot xmlns:xacro="http://www.ros.org/wiki/xacro">
-  <xacro:macro name="hokuyo_ust10" params="prefix mount update_rate:=50 sample_size:=720 min_angle:=-2.35619 max_angle:=2.35619 min_range:=0.1 max_range:=30.0 robot_namespace:=/ ">
+  <!-- ===================================================================
+       Hokuyo UST-10 LiDAR macro — Gazebo Harmonic version.
+       Gazebo Classic used libgazebo_ros_laser.so which embedded ROS
+       publishing directly in the plugin.
+       Gazebo Harmonic separates concerns:
+       1. The <sensor type="gpu_lidar"> block defines the physics/sim sensor.
+          It publishes on a gz topic (e.g. /front_laser/scan).
+       2. ros_gz_bridge (launched in gazebo.launch.py) bridges that gz topic
+          to a ROS2 sensor_msgs/msg/LaserScan topic of the same name.
+       The Sensors system plugin in automaton_world.sdf enables all sensors.
+       =================================================================== -->
+  <xacro:macro name="hokuyo_ust10" params="prefix mount update_rate:=50 sample_size:=720 min_angle:=-2.35619 max_angle:=2.35619 min_range:=0.1 max_range:=30.0 robot_namespace:=/">
     <link name="${prefix}_laser">
       <inertial>
-        <mass value="1.1" />
-        <origin xyz="0 0 0" />
-        <inertia ixx="${0.0833333 * 1.1 * (0.102*0.102 + 0.152*0.152)}" ixy="0.0" ixz="0.0"
+        <mass value="1.1"/>
+        <origin xyz="0 0 0"/>
+        <inertia
+          ixx="${0.0833333 * 1.1 * (0.102*0.102 + 0.152*0.152)}" ixy="0.0" ixz="0.0"
           iyy="${0.0833333 * 1.1 * (0.105*0.105 + 0.152*0.152)}" iyz="0.0"
-          izz="${0.0833333 * 1.1 * (0.105*0.105 + 0.102*0.102)}" />
+          izz="${0.0833333 * 1.1 * (0.105*0.105 + 0.102*0.102)}"/>
       </inertial>
       <visual>
         <origin xyz="0.0 0.0 0.0" rpy="0.0 0.0 0.0"/>
         <geometry>
-          <mesh filename="package://robot_description/meshes/hokuyo_ust10_lidar.stl" />
+          <mesh filename="package://robot_description/meshes/hokuyo_ust10_lidar.stl"/>
         </geometry>
-        <material name="dark_grey" />
+        <material name="dark_grey"/>
       </visual>
     </link>
@@ -23,11 +35,16 @@
       <origin xyz="0.0 0.0 0.007" rpy="0.0 0.0 0.0"/>
     </joint>
+    <!-- Gazebo Harmonic: gpu_lidar sensor.
+         Topic is published in the gz domain. The launch file bridges it to ROS2.
+         gz topic:  /${prefix}_laser/scan  (gz.msgs.LaserScan)
+         ROS2 topic: /${prefix}_laser/scan  (sensor_msgs/msg/LaserScan) -->
     <gazebo reference="${prefix}_laser">
-      <turnGravityOff>false</turnGravityOff>
-      <sensor type="ray" name="${prefix}_laser">
-        <pose>0 0 0 0 0 0</pose>
+      <material>Gazebo/DarkGrey</material>
+      <sensor name="${prefix}_lidar" type="gpu_lidar">
+        <topic>/${prefix}_laser/scan</topic>
+        <gz_frame_id>${prefix}_laser</gz_frame_id>
+        <update_rate>${update_rate}</update_rate>
         <visualize>false</visualize>
-        <update_rate>${update_rate}</update_rate>
-        <ray>
+        <lidar>
           <scan>
             <horizontal>
@@ -48,16 +65,7 @@
             <stddev>0.001</stddev>
           </noise>
-        </ray>
-        <plugin name="gazebo_ros_laser" filename="libgazebo_ros_laser.so">
-          <topicName>${prefix}_laser/scan</topicName>
-          <frameName>${prefix}_laser</frameName>
-          <robotNamespace>${robot_namespace}</robotNamespace>
-        </plugin>
+        </lidar>
+        <always_on>1</always_on>
       </sensor>
-    </gazebo>
-    <gazebo reference="${prefix}_laser">
-      <material>
-        Gazebo/DarkGrey
-      </material>
     </gazebo>
   </xacro:macro>

Commit message: feat(gazebo): add world selection and fix material warnings
World selection via launch argument:
  ros2 launch robot_description gazebo.launch.py world:=office
  ros2 launch robot_description gazebo.launch.py world:=warehouse
  ros2 launch robot_description gazebo.launch.py world:=construction
  ros2 launch robot_description gazebo.launch.py world:=orchard
  ros2 launch robot_description gazebo.launch.py world:=pipeline
  ros2 launch robot_description gazebo.launch.py world:=solar_farm
  ros2 launch robot_description gazebo.launch.py world:=empty  (default)
  ros2 launch robot_description gazebo.launch.py world:=/full/path/to/world.sdf

OpaqueFunction resolves short names to clearpath_gz world paths at launch
time. All clearpath worlds already include Sensors/Imu/NavSat plugins.

Also fix Ogre material script warnings:
  Gazebo/Red → SDF ambient/diffuse/specular RGBA colors (chassis)
  Gazebo/DarkGrey → SDF RGBA colors (lidar)

File: src/robot_description/urdf/laser.urdf.xacro (robot description, xacro)
@@ -40,5 +40,11 @@
          ROS2 topic: /${prefix}_laser/scan  (sensor_msgs/msg/LaserScan) -->
     <gazebo reference="${prefix}_laser">
-      <material>Gazebo/DarkGrey</material>
+      <visual>
+        <material>
+          <ambient>0.3 0.3 0.3 1</ambient>
+          <diffuse>0.3 0.3 0.3 1</diffuse>
+          <specular>0.1 0.1 0.1 1</specular>
+        </material>
+      </visual>
       <sensor name="${prefix}_lidar" type="gpu_lidar">
         <topic>/${prefix}_laser/scan</topic>
