Commit message: change chassis link to red

File: src/robot_description/urdf/automaton.urdf.xacro (robot description, xacro)
@@ -20,6 +20,6 @@
         <color rgba="0.4 0.4 0.4 1.0"/>
     </material>
-    <material name="yellow">
-        <color rgba="0.8 0.8 0.0 1.0"/>
+    <material name="Red">
+        <color rgba="0.8 0 0.0 1.0"/>
     </material>
     <material name="black">
@@ -87,5 +87,5 @@
                 <mesh filename="package://robot_description/meshes/base.stl"/>
             </geometry>
-            <material name="yellow" />
+            <material name="Red" />
         </visual>
         <collision>
@@ -113,4 +113,15 @@
         <origin xyz="${-wheel_base/2} ${-track_width/2} ${wheel_vertical_offset}" rpy="0.0 0.0 0.0"/>
     </xacro:wheel>
+    <link name="imu_link">
+      <interial>
+        <mass value="0.001"/>
+        <origin xyz="0 0 0" rpy="0 0 0" />
+        <inertia ixx="${dummy_inertia}" ixy="0.0" ixz="0.0" iyy="${dummy_inertia}" iyz="0.0" izz="${dummy_inertia}"/>
+      </interial>
+    </link>
+    <joint name="imu_joint" type="fixed">
+      <parent link="chassis_link"/>
+      <child link="imu_link"/>
+    </joint>
     <xacro:include filename="$(find robot_description)/urdf/automaton.gazebo" />
 </robot>

Commit message: add front mount and rear mount for the lasers

File: src/robot_description/urdf/automaton.urdf.xacro (robot description, xacro)
@@ -1,4 +1,6 @@
 <?xml version="1.0"?>
 <robot name="automaton" xmlns:xacro="http://www.ros.org/wiki/xacro">
+    <xacro:include filename="$(find robot_description)/urdf/automaton.gazebo" />
+    <xacro:include filename="$(find robot_description)/urdf/laser.urdf.xacro" />
     <xacro:property name="PI" value="3.14159"/>
     <xacro:property name="wheel_base" value="0.262"/>
@@ -124,4 +126,16 @@
       <child link="imu_link"/>
     </joint>
-    <xacro:include filename="$(find robot_description)/urdf/automaton.gazebo" />
+    <link name="front_mount"/>
+    <joint name="front_mount_joint" type="fixed">
+      <parent link="chassis_link"/>
+      <child link="front_mount"/>
+      <origin xyz="${chassis_length/2.2} 0.0 ${chassis_height}" rpy="0.0 0.0 0.0"/>
+    </joint>
+    <link name="rear_mount"/>
+    <joint name="rear_mount_joint" type="fixed">
+      <parent link="chassis_link"/>
+      <child link="rear_mount"/>
+      <origin xyz="${-chassis_length/2.2} 0.0 ${chassis_height}" rpy="0.0 0.0 0.0"/>
+    </joint>
+    <xacro:hokuyo_ust10 prefix="front" mount="front_mount"/>
 </robot>

Commit message: add rear scan and update rviz config

File: src/robot_description/urdf/automaton.urdf.xacro (robot description, xacro)
@@ -136,6 +136,7 @@
       <parent link="chassis_link"/>
       <child link="rear_mount"/>
-      <origin xyz="${-chassis_length/2.2} 0.0 ${chassis_height}" rpy="0.0 0.0 0.0"/>
+      <origin xyz="${-chassis_length/2.2} 0.0 ${chassis_height}" rpy="0.0 0.0 ${-PI}"/>
     </joint>
-    <xacro:hokuyo_ust10 prefix="front" mount="front_mount"/>
+    <xacro:hokuyo_ust10 prefix="front" mount="front_mount" />
+    <xacro:hokuyo_ust10 prefix="rear" mount="rear_mount" />
 </robot>

Commit message: stash old changes

File: src/robot_description/urdf/automaton.urdf.xacro (robot description, xacro)
@@ -49,5 +49,5 @@
             </inertial>
         </link>
-        <gazebo reference="${prefix}_wheel_link">
+        <!-- <gazebo reference="${prefix}_wheel_link">
             <material>
                 Gazebo/DarkGrey
@@ -59,5 +59,5 @@
             <kd value="1" />
             <fdir1 value="1 0 0 " />
-        </gazebo>
+        </gazebo> -->
         <joint name="${prefix}_wheel_joint" type="continuous">
             <xacro:insert_block name="blah"/>
@@ -66,5 +66,5 @@
             <axis xyz="0.0 1 0.0"/>
         </joint>
-        <transmission name="${prefix}_wheel_trans" >
+        <!-- <transmission name="${prefix}_wheel_trans" >
             <type>transmission_interface/SimpleTransmission</type>
             <joint name="${prefix}_wheel_joint">
@@ -75,5 +75,5 @@
                 <mechanicalReduction>1</mechanicalReduction>
             </actuator>
-        </transmission>
+        </transmission> -->
     </xacro:macro>
     <link name="base_link"></link>
@@ -115,5 +115,5 @@
         <origin xyz="${-wheel_base/2} ${-track_width/2} ${wheel_vertical_offset}" rpy="0.0 0.0 0.0"/>
     </xacro:wheel>
-    <link name="imu_link">
+    <!-- <link name="imu_link">
       <interial>
         <mass value="0.001"/>
@@ -121,9 +121,9 @@
         <inertia ixx="${dummy_inertia}" ixy="0.0" ixz="0.0" iyy="${dummy_inertia}" iyz="0.0" izz="${dummy_inertia}"/>
       </interial>
-    </link>
-    <joint name="imu_joint" type="fixed">
+    </link> -->
+    <!-- <joint name="imu_joint" type="fixed">
       <parent link="chassis_link"/>
       <child link="imu_link"/>
-    </joint>
+    </joint> -->
     <link name="front_mount"/>
     <joint name="front_mount_joint" type="fixed">
@@ -132,11 +132,11 @@
       <origin xyz="${chassis_length/2.2} 0.0 ${chassis_height}" rpy="0.0 0.0 0.0"/>
     </joint>
-    <link name="rear_mount"/>
+    <!-- <link name="rear_mount"/>
     <joint name="rear_mount_joint" type="fixed">
       <parent link="chassis_link"/>
       <child link="rear_mount"/>
       <origin xyz="${-chassis_length/2.2} 0.0 ${chassis_height}" rpy="0.0 0.0 ${-PI}"/>
-    </joint>
+    </joint> -->
     <xacro:hokuyo_ust10 prefix="front" mount="front_mount" />
-    <xacro:hokuyo_ust10 prefix="rear" mount="rear_mount" />
+    <!-- <xacro:hokuyo_ust10 prefix="rear" mount="rear_mount" /> -->
 </robot>

Commit message: feat: add 3D LiDAR, IMU, GPS, and magnetometer to robot
URDF / sensor model:
- lidar3d.urdf.xacro (new): VLP-16 style gpu_lidar, 16 channels ±15° vertical,
  360° horizontal, 512 samples, 10 Hz, range 0.5-100 m, σ=0.01 m noise
- automaton.urdf.xacro: enable IMU link/joint (was commented out, had typo
  <interial>→<inertial>); add GPS link on top-rear of chassis; add
  lidar3d_mount on top-centre; include lidar3d.urdf.xacro
- automaton.gazebo: enable IMU sensor (100 Hz, MEMS noise+bias model);
  add magnetometer sensor on imu_link (50 Hz, σ=1.3e-4 T); add GPS/NavSat
  sensor on gps_link (10 Hz, 1 m horizontal noise)

Bridge (gazebo.launch.py):
- /top_lidar_3d/points  PointCloud2   gz.msgs.PointCloudPacked
- /imu/data             Imu           gz.msgs.IMU
- /magnetometer         MagneticField gz.msgs.Magnetometer
- /gps/fix              NavSatFix     gz.msgs.NavSat

World SDF files (all 6):
- Add gz-sim-navsat-system and gz-sim-magnetometer-system plugins
  (required for GPS and magnetometer sensors to produce data)

File: src/robot_description/urdf/automaton.urdf.xacro (robot description, xacro)
@@ -3,4 +3,5 @@
     <xacro:include filename="$(find robot_description)/urdf/automaton.gazebo" />
     <xacro:include filename="$(find robot_description)/urdf/laser.urdf.xacro" />
+    <xacro:include filename="$(find robot_description)/urdf/lidar3d.urdf.xacro" />
     <xacro:property name="PI" value="3.14159"/>
     <xacro:property name="wheel_base" value="0.262"/>
@@ -115,15 +116,39 @@
         <origin xyz="${-wheel_base/2} ${-track_width/2} ${wheel_vertical_offset}" rpy="0.0 0.0 0.0"/>
     </xacro:wheel>
-    <!-- <link name="imu_link">
-      <interial>
+    <!-- IMU — mounted at chassis centre (internal sensor) -->
+    <link name="imu_link">
+      <inertial>
         <mass value="0.001"/>
-        <origin xyz="0 0 0" rpy="0 0 0" />
-        <inertia ixx="${dummy_inertia}" ixy="0.0" ixz="0.0" iyy="${dummy_inertia}" iyz="0.0" izz="${dummy_inertia}"/>
-      </interial>
-    </link> -->
-    <!-- <joint name="imu_joint" type="fixed">
+        <origin xyz="0 0 0" rpy="0 0 0"/>
+        <inertia ixx="${dummy_inertia}" ixy="0.0" ixz="0.0"
+                 iyy="${dummy_inertia}" iyz="0.0" izz="${dummy_inertia}"/>
+      </inertial>
+    </link>
+    <joint name="imu_joint" type="fixed">
       <parent link="chassis_link"/>
       <child link="imu_link"/>
-    </joint> -->
+      <origin xyz="0 0 ${chassis_height/2}" rpy="0 0 0"/>
+    </joint>
+    <!-- GPS — antenna on top-rear of chassis -->
+    <link name="gps_link">
+      <inertial>
+        <mass value="0.001"/>
+        <origin xyz="0 0 0" rpy="0 0 0"/>
+        <inertia ixx="${dummy_inertia}" ixy="0.0" ixz="0.0"
+                 iyy="${dummy_inertia}" iyz="0.0" izz="${dummy_inertia}"/>
+      </inertial>
+      <visual>
+        <origin xyz="0 0 0" rpy="0 0 0"/>
+        <geometry><cylinder radius="0.02" length="0.03"/></geometry>
+        <material name="dark_grey"/>
+      </visual>
+    </link>
+    <joint name="gps_joint" type="fixed">
+      <parent link="chassis_link"/>
+      <child link="gps_link"/>
+      <!-- Top surface of chassis, offset towards rear -->
+      <origin xyz="${-chassis_length/4} 0 ${chassis_height + 0.015}" rpy="0 0 0"/>
+    </joint>
+    <!-- 2D LiDAR front mount -->
     <link name="front_mount"/>
     <joint name="front_mount_joint" type="fixed">
@@ -132,11 +157,13 @@
       <origin xyz="${chassis_length/2.2} 0.0 ${chassis_height}" rpy="0.0 0.0 0.0"/>
     </joint>
-    <!-- <link name="rear_mount"/>
-    <joint name="rear_mount_joint" type="fixed">
+    <!-- 3D LiDAR mount — top-centre of chassis -->
+    <link name="lidar3d_mount"/>
+    <joint name="lidar3d_mount_joint" type="fixed">
       <parent link="chassis_link"/>
-      <child link="rear_mount"/>
-      <origin xyz="${-chassis_length/2.2} 0.0 ${chassis_height}" rpy="0.0 0.0 ${-PI}"/>
-    </joint> -->
-    <xacro:hokuyo_ust10 prefix="front" mount="front_mount" />
-    <!-- <xacro:hokuyo_ust10 prefix="rear" mount="rear_mount" /> -->
+      <child link="lidar3d_mount"/>
+      <origin xyz="0.0 0.0 ${chassis_height}" rpy="0.0 0.0 0.0"/>
+    </joint>
+    <!-- Sensors -->
+    <xacro:hokuyo_ust10 prefix="front" mount="front_mount"/>
+    <xacro:velodyne_vlp16 prefix="top" mount="lidar3d_mount"/>
 </robot>

Commit message: feat: add full sensor suite, SLAM world, and sensor position fixes
Sensors:
- 2D LiDAR repositioned to front-bottom-centre (z=0.05m) then restored
  to original front-top mount (z=chassis_height); 3D LiDAR raised to
  chassis_height+0.1m so it clears the 2D LiDAR on top-centre of robot
- Fix gpu_lidar 3D topic: was /top_lidar_3d/points (wrong — point cloud
  ends up on ${topic}/points); corrected to /top_lidar_3d so bridge
  receives PointCloudPacked on /top_lidar_3d/points as intended

Worlds:
- Add <spherical_coordinates> to all 6 world SDF files; required by
  Gazebo Harmonic for GPS (NavSat) and Magnetometer sensors — without it
  both sensors fail with "Spherical coordinates not set" every physics tick
- Add slam_district.sdf: large 5-zone SLAM benchmark world (260×260 m)
  with pillar forest, industrial corridor, aliasing residential grid,
  sculptural park, and a 25m global landmark tower; ~13 min perimeter loop

Launch:
- Register slam_district in _WORLDS dict; refactor _resolve_world to map
  short names to filenames (cleaner than None sentinel + hardcoded fallback)
- Add slam_district to world:= docstring and argument description

README:
- Document all 5 sensors with topics, rates, and noise parameters
- Update architecture diagram and topic bridge map with new sensor topics
- Add world selection table and slam_district zone/design summary
- Update Phase 1 checklist to reflect completed sensor and world work

File: src/robot_description/urdf/automaton.urdf.xacro (robot description, xacro)
@@ -157,10 +157,10 @@
       <origin xyz="${chassis_length/2.2} 0.0 ${chassis_height}" rpy="0.0 0.0 0.0"/>
     </joint>
-    <!-- 3D LiDAR mount — top-centre of chassis -->
+    <!-- 3D LiDAR mount — centre of robot, raised above 2D lidar -->
     <link name="lidar3d_mount"/>
     <joint name="lidar3d_mount_joint" type="fixed">
       <parent link="chassis_link"/>
       <child link="lidar3d_mount"/>
-      <origin xyz="0.0 0.0 ${chassis_height}" rpy="0.0 0.0 0.0"/>
+      <origin xyz="0.0 0.0 ${chassis_height + 0.1}" rpy="0.0 0.0 0.0"/>
     </joint>
     <!-- Sensors -->

File: src/robot_description/urdf/lidar3d.urdf.xacro (robot description, xacro)
@@ -64,5 +64,8 @@
       </visual>
       <sensor name="${prefix}_3d_lidar" type="gpu_lidar">
-        <topic>/${prefix}_lidar_3d/points</topic>
+        <!-- Gazebo Harmonic publishes LaserScan on this topic,
+             and PointCloudPacked on ${topic}/points automatically.
+             Bridge entry in gazebo.launch.py subscribes to /${prefix}_lidar_3d/points. -->
+        <topic>/${prefix}_lidar_3d</topic>
         <gz_frame_id>${prefix}_lidar_3d_link</gz_frame_id>
         <update_rate>${update_rate}</update_rate>
